File: MP2905.kicad_pcb (KiCad board)
At the start: 2 copper layers, 15 parts, among them J1 Conn_01x04_Pin, Q1 NMOS, Q2 NMOS, Q3 NMOS, U1 MP2905EK-LF-P

Commit message: 二层板
Parts:
- removed J1: Conn_01x04_Pin, Connector_PinHeader_2.54mm:PinHeader_1x04_P2.54mm_Vertical
- removed the R1 at (96.8, 97.8)
- removed the R1 at (96.8, 102.8)
- added C10: C_1206, PCM_Capacitor_SMD_AKL:C_1206_3216Metric, F.Cu at (98.1, 78.1)
- added C11: CP_SMD_D10.0mm_H7.7mm, PCM_Capacitor_SMD_AKL:CP_Elec_10x7.7, F.Cu at (98.3, 71.5)
- added C12: C_0603, PCM_Capacitor_SMD_AKL:C_0603_1608Metric, F.Cu at (98.3, 65.2)
- added C13: 100nF, Capacitor_SMD:C_0603_1608Metric, F.Cu at (96.5, 49.5)
- added C14: 22nF, Capacitor_SMD:C_0603_1608Metric, F.Cu at (88.2, 47.3)
- added C15: 1μF, Capacitor_SMD:C_0603_1608Metric, F.Cu at (85.1, 48.0)
- added C5: CP_SMD_D10.0mm_H7.7mm, PCM_Capacitor_SMD_AKL:CP_Elec_10x7.7, F.Cu at (79.2, 71.5)
- added C6: C_0603, PCM_Capacitor_SMD_AKL:C_0603_1608Metric, B.Cu at (79.4, 67.4)
- added C7: C_1206, PCM_Capacitor_SMD_AKL:C_1206_3216Metric, B.Cu at (79.3, 73.6)
- added C8: C_1206, PCM_Capacitor_SMD_AKL:C_1206_3216Metric, B.Cu at (79.3, 70.3)
- added C9: C_1206, PCM_Capacitor_SMD_AKL:C_1206_3216Metric, B.Cu at (98.1, 78.1)
- added D1: 1N4148WS, PCM_Diode_SMD_AKL:D_SOD-323, F.Cu at (103.2, 51.0)
- added R1: R, Resistor_SMD:R_0603_1608Metric, F.Cu at (89.8, 47.3)
- added R5: 20R, Resistor_SMD:R_0603_1608Metric, F.Cu at (103.2, 49.0)
- added R6: 3K, Resistor_SMD:R_0603_1608Metric, F.Cu at (85.1, 46.5)
- added SW1: SW_Nidec_CAS-120A1, 自建封装库:SW-TH_SHOU-HAN_SS12D10G4, F.Cu at (71.2, 53.6)
- L1: moved to F.Cu
- moved Q3 75.0 mm to (77.6, 48.1), turned to -90 degrees
- moved R3 53.3 mm to (91.3, 47.3), turned to 90 degrees
- moved U1 53.2 mm to (92.0, 51.0)
- moved R4 50.5 mm to (76.7, 51.8), turned to 180 degrees
- moved R2 50.1 mm to (94.0, 48.1)
- moved C4 49.1 mm to (94.0, 46.6)
- moved Q1 46.9 mm to (102.7, 55.6)
- moved Q2 46.8 mm to (100.8, 61.6)
- moved C2 46.7 mm to (84.3, 50.3), turned to -90 degrees
- moved L1 44.9 mm to (108.6, 54.1)
- moved C1 44.4 mm to (86.6, 49.5)
- moved C3 40.8 mm to (96.5, 52.8), turned to 90 degrees
Connections:
- Q1 pad 2: /HG -> Net-(D1-A)
Routing:
- net GND: track 0.00 -> 100.5 mm, vias 0 -> 26
- net /VOUT: track 0.00 -> 48.1 mm, vias 0 -> 26
- net /LG: track 0.00 -> 21.5 mm, vias 0 -> 2
- net /SW: track 0.00 -> 17.8 mm, vias 59 -> 35
- net Net-(Q3-D): track 0.00 -> 13.5 mm
- net +12V: track 0.00 -> 10.6 mm, vias 0 -> 61
- net Net-(U1-FB): track 0.00 -> 7.39 mm
- net /EN: track 0.00 -> 7.27 mm
- net Net-(U1-REF): track 0.00 -> 5.41 mm
- net Net-(D1-A): track 0.00 -> 5.14 mm
- net Net-(U1-ILIM): track 0.00 -> 4.33 mm
- net Net-(U1-BST): track 0.00 -> 2.92 mm
- net Net-(C14-Pad1): track 0.00 -> 2.29 mm
- net /HG: track 9.22 -> 10.1 mm
- added copper zone on B.Cu, net +12V
- added copper zone on F.Cu, net +12V
- added copper zone on B.Cu, net /VOUT
- added copper zone on F.Cu, net /VOUT
- added copper zone on B.Cu, net GND
- added copper zone on F.Cu, net GND
Other:
- board outline added: 45 x 36.5 mm
- board text added: "{ "ViaStitching": "0.2", "stitch_zone_0": { "HSpacing": "1.5", "VSpacing": "1.5", "HOffset": "1", "VOffset": "1", "Clearance": "0", "Randomize": false } }"
- board text added: "{ "ViaStitching": "0.2", "stitch_zone_0": { "HSpacing": "2", "VSpacing": "2", "HOffset": "1", "VOffset": "1", "Clearance": "0", "Randomize": false } }"

Commit message: 四层板
Parts:
- removed C12: C_0603, PCM_Capacitor_SMD_AKL:C_0603_1608Metric
- C10: value C_1206 -> 100UF
- C11: value CP_SMD_D10.0mm_H7.7mm -> 470uF
- C5: value CP_SMD_D10.0mm_H7.7mm -> 470UF
- C6: value C_0603 -> 10NF; moved to F.Cu
- C7, C8: value C_1206 -> 4.7UF; moved to F.Cu
- C9: value C_1206 -> 100UF; moved to F.Cu
- L1: moved to B.Cu
- R1: value R -> 1K
- R3: value R -> 2K
- R4: value R -> 20K
- R6: value 3K -> 10R
- moved Q3 62.4 mm to (91.2, 109.0), turned to 90 degrees
- moved R4 60.5 mm to (94.8, 109.5), turned to 90 degrees
- moved C2 60.4 mm to (96.3, 109.5), turned to 90 degrees
- moved C4 60.0 mm to (104.6, 105.7)
- moved C8 59.6 mm to (91.3, 128.7)
- moved R6 59.4 mm to (96.3, 104.9), turned to 90 degrees
- moved R1 58.6 mm to (100.8, 104.9)
- moved R3 58.6 mm to (102.2, 104.9)
- moved C15 58.6 mm to (99.3, 104.9), turned to -90 degrees
- moved U1 58.5 mm to (101.2, 108.8)
- moved C14 58.4 mm to (97.8, 104.9)
- moved C1 58.3 mm to (95.5, 107.2)
- moved C3 58.2 mm to (106.0, 110.2)
- moved R2 57.0 mm to (104.6, 104.1)
- moved C13 56.4 mm to (107.0, 104.9)
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Routing:
- net GND: track 100.5 -> 10.2 mm, vias 26 -> 54
- net /VOUT: track 48.1 -> 23.8 mm, vias 26 -> 37
- net /HG: track 10.1 -> 27.9 mm
- net /LG: track 21.5 -> 13.1 mm, vias 2 -> 0
- net /SW: track 17.8 -> 25.9 mm, vias 35 -> 16
- net Net-(U1-REF): track 5.41 -> 2.73 mm
- net +12V: track 10.6 -> 8.11 mm, vias 61 -> 52
- net Net-(D1-A): track 5.14 -> 3.42 mm
- net Net-(C14-Pad1): track 2.29 -> 1.52 mm
- net Net-(U1-FB): track 7.39 -> 6.72 mm
- net Net-(Q3-D): track 13.5 -> 13.4 mm, vias 0 -> 2
- added copper zone on In1.Cu, net +12V
- added copper zone on In2.Cu, net +12V
- added copper zone on In1.Cu, net /SW
- added copper zone on In2.Cu, net /SW
- added copper zone on In1.Cu, net /VOUT
- added copper zone on In2.Cu, net /VOUT
- added copper zone on In1.Cu, net GND
- added copper zone on In2.Cu, net GND
Other:
- board size 45 x 36.5 mm -> 60 x 35 mm
- copper layers 2 -> 4
