File: MP2905.kicad_sch (KiCad schematic)
At the start: 13 parts, among them Q1 NMOS, Q2 NMOS, Q3 NMOS, U1 MP2905EK-LF-P

Commit message: 二层板
Parts:
- added C10, C7, C8, C9: C_1206, PCM_Capacitor_SMD_AKL:C_1206_3216Metric, symbol PCM_Capacitor_AKL:C_1206
- added C11, C5: CP_SMD_D10.0mm_H7.7mm, PCM_Capacitor_SMD_AKL:CP_Elec_10x7.7, symbol PCM_Capacitor_AKL:CP_SMD_D10.0mm_H7.7mm
- added C12, C6: C_0603, PCM_Capacitor_SMD_AKL:C_0603_1608Metric, symbol PCM_Capacitor_AKL:C_0603
- added C13: 100nF, Capacitor_SMD:C_0603_1608Metric, symbol Device:C
- added C14: 22nF, Capacitor_SMD:C_0603_1608Metric, symbol Device:C
- added C15: 1μF, Capacitor_SMD:C_0603_1608Metric, symbol Device:C
- added D1: 1N4148WS, PCM_Diode_SMD_AKL:D_SOD-323, symbol PCM_Diode_AKL:1N4148WS
- added R5: 20R, Resistor_SMD:R_0603_1608Metric, symbol Device:R
- added R6: 3K, Resistor_SMD:R_0603_1608Metric, symbol Device:R
- added SW1: SW_Nidec_CAS-120A1, 自建封装库:SW-TH_SHOU-HAN_SS12D10G4, symbol Switch:SW_Nidec_CAS-120A1
Connections:
- net +12V: now also C13.2, C5.1, C6.1, C7.1, C8.1, SW1.2 (B), SW1.3 (A)
- net EN: now also SW1.1 (C)
- net GND: now also C10.2, C11.2, C12.2, C13.1, C15.1, C5.2, C6.2, C7.2, C8.2, C9.2
- net HG: now also D1.1 (K), R5.2; no longer Q1.2 (G)
- net VOUT: now also C10.1, C11.1, C12.1, C9.1, R6.1
- net at R1.2, R3.1, U1.1 (FB): now also C14.2, C15.2
- new net: D1.2 (A), Q1.2 (G), R5.1
- new net: C14.1, R6.2
Other:
- moved on the sheet: R3

Commit message: 四层板
Parts:
- removed C12: C_0603, PCM_Capacitor_SMD_AKL:C_0603_1608Metric, symbol PCM_Capacitor_AKL:C_0603
- C10, C9: value C_1206 -> 100UF
- C11: value CP_SMD_D10.0mm_H7.7mm -> 470uF
- C5: value CP_SMD_D10.0mm_H7.7mm -> 470UF
- C6: value C_0603 -> 10NF
- C7, C8: value C_1206 -> 4.7UF
- R1: value R -> 1K
- R3: value R -> 2K
- R4: value R -> 20K
- R6: value 3K -> 10R
Changed lines of the file:
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@@
 			"FNKK8oJZ1jzyD13bl3U4agGRO4iW66DLfKXiQL4fN2AusgmNcsPs6WnOPH17zuqrjokkZ2jzyTnz"
 			"9DP8V+pyRJyhmJGb5ixn2GM+aXqPkgp35CKOLMuRcaUa8AVPMp8vq6Nx3bFDC+YZ6GNWDcQ6bPka"
-			"B2LMlq+hlF0TdAdpDZKX78gdVZAtWl8nYjjDTEIn+lqEQx/ZAA=="
+			"B2LMlq+hlF0TdAdpDZKX78gdVZAtWl8nYjjDTEIn+lqEQx/ZAAAAAAAAAAAAAAAAAAAAAAAAAAAA"
+			"AAAAAAAAAAAAAAAAAAAAAAAAAAAAAAAAAAAAAAAAAAAAAAAAAAAAAAAAAAAAAAAAAAAAAAAAAAAA"
+			"AAAAAAAAAAAAAAAAAAAAAAAAAAAAAAAAAAAAAAAAAAAAAAAAAAAAAAAAAAAAAAAAAAAAAAAAAAAA"
+			"AAAAAAAAAAAAAAAAAAAAAAAAAAAAAAAAAAAAAAAAAAAAAAAAAAAAAAAAAAAAAAAAAAAAAAAAAAAA"
+			"AAAAAAAAAAAAAAAAAAAAAAAAAAAAAAAAAAAAAAAAAAAAAAAAAAAAAAAAAAAAAAAAAAAAAAAAAAAA"
+			"AAAAAAAAAAAAAAAAAAAAAAAAAAAAAAAAAAAAAAAAAAAAAAAAAAAAAAAAAAAAAAAAAAAAAAAAAAAA"
+			"AAAAAAAAAAAAAAAAAAAAAAAAAAAAAAAAAAAAAAAAAAAAAAAAAAAAAAAAAAAAAAAAAAAAAAAAAAAA"
+			"AAAAAAAAAAAAAAAAAAAAAAAAAAAAAAAAAAAAAAAAAAAAAAAAAAAAAAAAAAAAAAAAAAAAAAAAAAAA"
+			"AAAAAAAAAAAAAAAAAAAAAAAAAAAAAAAAAAAAAAAAAAAAAAAAAAAAAAAAAAAAAAAAAAAAAAAAAAAA"
+			"AAAAAAAAAAAAAAAAAAAAAAAAAAAAAAAAAAAAAAAAAAAAAAAAAAAAAAAAAAAAAAAAAAAAAAAAAAAA"
+			"AAAAAAAAAAAAAAAAAAAAAAAAAAAAAAAAAAAAAAAAAAAAAAAAAAAAAAAAAAAAAAAAAAAAAAAAAAAA"
+			"AAAAAAAAAAAAAAAAAAAAAAAAAAAAAAAAAAAAAAAAAAAAAAAAAAAAAAAAAAAAAAAAAAAAAAAAAAAA"
+			"AAAAAAAAAAAAAAAAAAAAAAAAAAAAAAAAAAAAAAAAAAAAAAAAAAAAAAAAAAAAAAAAAAAAAAAAAAAA"
+			"AAAAAAAAAAAAAAAAAAAAAAAAAAAAAAAAAAAAAAAAAAAAAAAAAAAAAAAAAAAAAAAAAAAAAAAAAAAA"
+			"AAAAAAAAAAAAAAAAAAAAAAAAAAAAAAAAAAAAAAAAAAAAAAAAAAAAAAAAAAAAAAAAAAAAAAAAAAAA"
+			"AAAAAAAAAAAAAAAAAAAAAAAAAAAAAAAAAAAAAAAAAAAAAAAAAAAAAAAAAAAAAAAAAAAAAAAAAAAA"
+			"AAAAAAAAAAAAAAAAAAAAAAAAAAAAAAAAAAAAAAAAAAAAAAAAAAAAAAAAAAAAAAAAAAAAAAAAAAAA"
+			"AAAAAAAAAAAAAAAAAAAAAAAAAAAAAAAAAAAAAAAAAAAAAAAAAAAAAAAAAAAAAAAAAAAAAAAAAAAA"
+			"AAAAAAAAAAAAAAAAAAAAAAAAAAAAAAAAAAAAAAAAAAAAAAAAAA=="
 		)
 	)
@@
 			"S2U5N3puOFhqT091c3N6ajMzWE43KzlyZnpneC84Z0UyYk5nRXdhZW5TcFZ4NzdiVTBOallDOE8v"
 			"MndoZStrUFBQUDU4Z0NQamtKei9KNXovL2VRRDI1WkZISHVIRUUwK2t2NytmbDcvODVmejJ0Ny9G"
-			"R0FQQWs5SGYzOCtXTFZzQVNDeGR1aFFBbA=="
+			"R0FQQWs5SGYzOCtXTFZzQVNDeGR1aFFBbAA0ADIAWQB0AGYAegBNAFQARQBCAEoAZABlAGMAZwBr"
+			"AHYAZQAvAEcATABBAFoAagAwAGkAMQAvADkAaQBsAG0AegBaAG4ASAA2AEcAVwBmAHcAdQB0AGUA"
+			"LwBIAG8AQwAvAFgAbgBRAFIATAAzAHYAeABpADgAbgBuADgAMQB4ADYAeQBTAFcAOAA3AE0AVQB2"
+			"AFoAbQArAEgASABYAFkAWQA5AFEAMABOAEEASAB6ACsAYwA1AC8AagBaAFMAOQArAE0AUgBNAFQA"
+			"RQAzAHoAcABpADEALwBrAFoAUwA5ACsATQBRAEQALwBIADMAMwArAGMANQAvAGoAWgBTADkAKwBN"
+			"AFIATQBUAEUAMwB6AHAAaQAxAC8AawBaAFMAOQArAE0AUQBDAEoAdgAxADUAMABFAFMAOQA3ADgA"
+			"WQB1ADUAOQBKAEoATAA2AE8AdgByADQAMgBVAHYAZgBqAEYALwB2AGUAZwBpAEEAQwBaADkALwBn"
+			"AHQAZgA0AEgAZAAvACsAQQBOAFgAWABIADQANQByADMAcgA1AHkANwBuAHoAegBqAHQANQA5ADMA"
+			"dgBmAHkAMgB0AGYALwAzAHIAbQB6AFoAcwBIAGcATQB1AGUAagBJAGEARwBCAGcANAA0ADgARQBD"
+			"ADYAdQByAHQAcABhAEcAZwBBADQAUABHADgAOQBuAFcAdgA0ADcAWgBiAGIAKwBXADEAcgAzAHMA"
+			"ZABBAEkAOQBuADYAdABTAHAASABIAGIANAA0AGIAegAyADkAYQA4AEgAdwBHAFYAUAB4AGUAYwAv"
+			"ADkAegBrAEEAWABPAGEAeQAvADYAUwB4AHMAVABHACsAKwA1ADMAdgA4AE4AdwB6AHoAZwBEAGcA"
+			"MABpAHUAdQA0AE4AMwB2AGUAUQA4AE4ARABRADAAQQBQAEYAMABmAGYAUAAvADcAQQBmAGoANgBO"
+			"ADcAOABKAHcATwBQAFoAcwBXAE0ASABBAEgAdgA3ADkAYQA5ACsAeABRAHYAUABQAFoAZQBHAGgA"
+			"ZwBZAEEAOQB1AFoANQBIAGcAQwBUAEcAaABvAGEAKwBQAG8AMwB2ADgAbABiADMAdgBoAEcAQQBQ"
+			"ADcAYgBqAFkAMgBOADgAZAAzAHYAZgBJAGYAbgBuAG4ARQBHAEEASAA4ADYALwAzAHoAZQAvAFoA"
+			"NwAzADAATgBEAFEAQQBNAEQAVAA5AGUASwBYAHYASQBTAFYAQgB4AHoAQQA1AHoALwAzAE8AVgBh"
+			"AHQAVwBzAFcATwBIAFQAdgA0ADcAbgBlACsAdwArAHIASABIAHUATwBGAEwAMwBvAFIAQQBDADUA"
+			"egBtAGMAdABjADUAagBLAFgALwBYADkAaw=="
 		)
 	)
@@
 			)
 		)
-		(property "Value" "C_1206"
+		(property "Value" "100UF"
 			(at 238.76 59.6899 0)
 			(effects
@@
 			)
 		)
-		(property "Value" "R"
+		(property "Value" "1K"
 			(at 77.47 49.53 90)
 			(effects
@@
 			)
 		)
-		(property "Value" "C_1206"
+		(property "Value" "100UF"
 			(at 233.68 59.6899 0)
 			(effects
@@
 	)
 	(symbol
-		(lib_id "PCM_Capacitor_AKL:C_0603")
-		(at 245.11 58.42 0)
-		(unit 1)
-		(exclude_from_sim no)
-		(in_bom yes)
-		(on_board yes)
-		(dnp no)
-		(property "Reference" "C12"
-			(at 246.38 55.88 0)
-			(effects
-				(font
-					(size 1.27 1.27)
-				)
-				(justify left)
-			)
-		)
-		(property "Value" "C_0603"
-			(at 248.92 59.6899 0)
-			(effects
-				(font
-					(size 1.27 1.27)
-				)
-				(justify left)
-				(hide yes)
-			)
-		)
-		(property "Footprint" "PCM_Capacitor_SMD_AKL:C_0603_1608Metric"
-			(at 246.0752 62.23 0)
-			(effects
-				(font
-					(size 1.27 1.27)
-				)
-				(hide yes)
-			)
-		)
-		(property "Datasheet" "~"
-			(at 245.11 58.42 0)
-			(effects
-				(font
-					(size 1.27 1.27)
-				)
-				(hide yes)
-			)
-		)
-		(property "Description" "SMD 0603 MLCC capacitor, Alternate KiCad Library"
-			(at 245.11 58.42 0)
-			(effects
-				(font
-					(size 1.27 1.27)
-				)
-				(hide yes)
-			)
-		)
-		(pin "1"
-		)
-		(pin "2"
-		)
-		(instances
-			(project "MP2905"
-				(path "/84bd166f-0dbb-4308-81e7-3ed364f48bde"
-					(reference "C12")
-					(unit 1)
-				)
-			)
-		)
-	)
-	(symbol
 		(lib_id "power:GND")
 		(at 50.8 72.39 0)
@@
 			)
 		)
-		(property "Value" "CP_SMD_D10.0mm_H7.7mm"
+		(property "Value" "470UF"
 			(at 48.26 30.8609 0)
 			(effects
@@
 			)
 		)
-		(property "Value" "R"
+		(property "Value" "20K"
 			(at 82.55 76.2 90)
 			(effects
@@
 			)
 		)
-		(property "Value" "CP_SMD_D10.0mm_H7.7mm"
+		(property "Value" "470uF"
 			(at 243.84 58.8009 0)
 			(effects
@@
 			)
 		)
-		(property "Value" "C_1206"
+		(property "Value" "4.7UF"
 			(at 43.18 31.7499 0)
 			(effects
@@
 			)
 		)
-		(property "Value" "3K"
+		(property "Value" "10R"
 			(at 135.636 25.908 90)
 			(effects
@@
 			)
 		)
-		(property "Value" "R"
+		(property "Value" "2K"
 			(at 134.62 36.83 90)
 			(effects
@@
 			)
 		)
-		(property "Value" "C_0603"
+		(property "Value" "10NF"
 			(at 53.34 31.7499 0)
 			(effects
@@
 			)
 		)
-		(property "Value" "C_1206"
+		(property "Value" "4.7UF"
 			(at 38.1 31.7499 0)
 			(effects
